Commit message: Updated project files

File: src/bot_description/urdf/bot.urdf.xacro (robot description, xacro)
@@ -172,5 +172,5 @@
     <parent link="base_link"/>
     <child link="camera_mount_link"/>
-    <origin xyz="0.345 0 0.15" rpy="0 -0.15 0"/>
+    <origin xyz="0.345 0 0.15" rpy="0 -0.05 0"/>
   </joint>
   <link name="camera_link">

File: src/bot_description/urdf/bot_wheel.urdf.xacro (robot description, xacro)
@@ -44,5 +44,5 @@
 		<gazebo reference="${wheel_prefix}_wheel_link">
 			<mu1>1.0</mu1>
-			<mu2>0.2</mu2>
+			<mu2>0.4</mu2>
 			<kp>10000000.0</kp>
 			<kd>1.0</kd>
